File: PCBs/SensorNivel/sensor_dsp.sch (EAGLE design)
At the start: 76 parts, among them IC1 LD117AS, IC2 DSPIC33FJ12GP202/SP, IC4 7805TV, IC5 ICL7660CPA, IC6 4069N, IC7 LM324N, IC8 LM324N, IC9 MAX481CPA

Commit message: Se hicieron modificaciones al Firmware y al Software. Version funcional.
Parts:
- C1, C2: value (none) -> 22pF
- C10, C11, C12, C25, C26, C27, C28: value (none) -> 100nF
- C3, C4, C5: value (none) -> 10nF
- C6, C7, C8: value (none) -> 1nF
- C9: value (none) -> 10uF
- Q6: value (none) -> 8MHz
- R12, R13: value (none) -> 4.7K
- R14, R15, R20, R28, R29, R30, R31, R32, R33, R34: value (none) -> 10K
- R16: value (none) -> 1M
- R17, R25: value (none) -> 1K
- R18, R26, R27: value (none) -> 3.3K
- R19: value (none) -> 470
- R2: value (none) -> 120
- R21: value (none) -> 390
- R22, R23: value (none) -> 220
- R35, R36: value (none) -> 2.2K
